Commit message: sinusoidal test

File: robot3.urdf (robot description, URDF)
Before this commit: robot hexapod, 25 links, 24 joints
Links:
- link BLH: geometry collision box size=1.0 0.3 0.3; visual mesh filename=package://crab_description/meshes/femur_l.STL scale=10 10 10
- link BLK: geometry collision box size=0.1 0.1 1.0; visual mesh filename=package://crab_description/meshes/tibia_l.STL scale=10 10 10
- link BLP: geometry collision box size=0.05 0.05 0.05; visual mesh filename=package://crab_description/meshes/coxa_l.STL scale=10 10 10
- link BRH: geometry collision box size=1.0 0.3 0.3; visual mesh filename=package://crab_description/meshes/femur_r.STL scale=10 10 10
- link BRK: geometry collision box size=0.1 0.1 1.0; visual mesh filename=package://crab_description/meshes/tibia_r.STL scale=10 10 10
- link BRP: geometry collision box size=0.05 0.05 0.05; visual mesh filename=package://crab_description/meshes/coxa_r.STL scale=10 10 10
- link FLH: geometry collision box size=1.0 0.3 0.3; visual mesh filename=package://crab_description/meshes/femur_l.STL scale=10 10 10
- link FLK: geometry collision box size=0.1 0.1 1.0; visual mesh filename=package://crab_description/meshes/tibia_l.STL scale=10 10 10
- link FLP: geometry collision box size=0.05 0.05 0.05; visual mesh filename=package://crab_description/meshes/coxa_l.STL scale=10 10 10
- link FRH: geometry collision box size=1.0 0.3 0.3; visual mesh filename=package://crab_description/meshes/femur_r.STL scale=10 10 10
- link FRK: geometry collision box size=0.1 0.1 1.0; visual mesh filename=package://crab_description/meshes/tibia_r.STL scale=10 10 10
- link FRP: geometry collision box size=0.05 0.05 0.05; visual mesh filename=package://crab_description/meshes/coxa_r.STL scale=10 10 10
- link MLH: geometry collision box size=1.0 0.3 0.3; visual mesh filename=package://crab_description/meshes/femur_l.STL scale=10 10 10
- link MLK: geometry collision box size=0.1 0.1 1.0; visual mesh filename=package://crab_description/meshes/tibia_l.STL scale=10 10 10
- link MLP: geometry collision box size=0.05 0.05 0.05; visual mesh filename=package://crab_description/meshes/coxa_l.STL scale=10 10 10
- link MRH: geometry collision box size=1.0 0.3 0.3; visual mesh filename=package://crab_description/meshes/femur_r.STL scale=10 10 10
- link MRK: geometry collision box size=0.1 0.1 1.0; visual mesh filename=package://crab_description/meshes/tibia_r.STL scale=10 10 10
- link MRP: geometry collision box size=0.05 0.05 0.05; visual mesh filename=package://crab_description/meshes/coxa_r.STL scale=10 10 10

Commit message: new tripod evolution

File: robot3.urdf (robot description, URDF)
Before this commit: robot hexapod, 25 links, 24 joints
Links:
- link BLH: geometry collision box size=0.4 0.1 0.3; visual mesh filename=package://crab_description/meshes/femur_l.STL scale=10 10 10
- link BLP: geometry collision box size=0.1 0.1 0.1; visual mesh filename=package://crab_description/meshes/coxa_l.STL scale=10 10 10
- link BRH: geometry collision box size=0.4 0.1 0.3; visual mesh filename=package://crab_description/meshes/femur_r.STL scale=10 10 10
- link BRP: geometry collision box size=0.1 0.1 0.1; visual mesh filename=package://crab_description/meshes/coxa_r.STL scale=10 10 10
- link FLH: geometry collision box size=0.4 0.1 0.3; visual mesh filename=package://crab_description/meshes/femur_l.STL scale=10 10 10
- link FLP: geometry collision box size=0.1 0.1 0.1; visual mesh filename=package://crab_description/meshes/coxa_l.STL scale=10 10 10
- link FRH: geometry collision box size=0.4 0.1 0.3; visual mesh filename=package://crab_description/meshes/femur_r.STL scale=10 10 10
- link FRP: geometry collision box size=0.1 0.1 0.1; visual mesh filename=package://crab_description/meshes/coxa_r.STL scale=10 10 10
- link MLH: geometry collision box size=0.4 0.1 0.3; visual mesh filename=package://crab_description/meshes/femur_l.STL scale=10 10 10
- link MLP: geometry collision box size=0.1 0.1 0.1; visual mesh filename=package://crab_description/meshes/coxa_l.STL scale=10 10 10
- link MRH: geometry collision box size=0.4 0.1 0.3; visual mesh filename=package://crab_description/meshes/femur_r.STL scale=10 10 10
- link MRP: geometry collision box size=0.1 0.1 0.1; visual mesh filename=package://crab_description/meshes/coxa_r.STL scale=10 10 10
